File: esp32 switch.kicad_pcb (KiCad board)
At the start: 2 copper layers, 88.9 x 55.9 mm, 26 parts, among them J1 Screw_Terminal_01x04, J2 Screw_Terminal_01x03, J3 Conn_02x07_Odd_Even, J5 Conn_01x06_Female, J6 Conn_01x07_Male, K1 Relay, K2 Relay, K3 Relay, K4 Relay, Q1 BC847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

Commit message: new
Parts:
- J1: value Screw_Terminal_01x04 -> Screw_Terminal_01x03; footprint TerminalBlock:TerminalBlock_Altech_AK300-4_P5.00mm -> TerminalBlock:TerminalBlock_Altech_AK300-3_P5.00mm
- moved J1 2.54 mm to (170.4, 101.6)
Connections:
- J1 pad 3: Earth -> AC
Routing:
- net Earth: track 190.1 -> 174.7 mm
- net Net-(K1-PadNO): track 12.4 -> 15.8 mm
- net AC: track 12.0 -> 14.9 mm
- net Net-(K2-PadNO): track 33.2 -> 35.6 mm
Other:
- board text added: "Mohammed Aslam NK"
