File: esp32 switch.kicad_sch (KiCad schematic)
At the start: 26 parts, among them J1 Screw_Terminal_01x04, J2 Screw_Terminal_01x03, J3 Conn_02x07_Odd_Even, J5 Conn_01x06_Female, J6 Conn_01x07_Male, K1 Relay, K2 Relay, K3 Relay, K4 Relay, Q1 BC847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

Commit message: new
Parts:
- removed J1: Screw_Terminal_01x04, TerminalBlock:TerminalBlock_Altech_AK300-4_P5.00mm, symbol Connector:Screw_Terminal_01x04
- added J1: Screw_Terminal_01x03, TerminalBlock:TerminalBlock_Altech_AK300-3_P5.00mm, symbol Connector:Screw_Terminal_01x03
Connections:
- net AC: now also J1.3 (Pin_3)
- net at K1.NO: now also J1.1 (Pin_1)
- net at K2.NO: now also J1.2 (Pin_2)
Changed lines of the file:
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@@
   (junction (at 48.26 82.55) (diameter 0) (color 0 0 0 0)
-  )
-  (junction (at 27.94 72.39) (diameter 0) (color 0 0 0 0)
   )
   (junction (at 266.7 72.39) (diameter 0) (color 0 0 0 0)
@@
     (stroke (width 0) (type default) (color 0 0 0 0))
   )
-  (wire (pts (xy 27.94 64.77) (xy 27.94 72.39))
+  (wire (pts (xy 27.94 64.77) (xy 27.94 87.63))
     (stroke (width 0) (type default) (color 0 0 0 0))
   )
@@
     (stroke (width 0) (type default) (color 0 0 0 0))
   )
-  (wire (pts (xy 17.78 74.93) (xy 20.32 74.93))
+  (wire (pts (xy 17.78 72.39) (xy 20.32 72.39))
     (stroke (width 0) (type default) (color 0 0 0 0))
   )
@@
     (stroke (width 0) (type default) (color 0 0 0 0))
   )
-  (wire (pts (xy 20.32 15.24) (xy 20.32 74.93))
+  (wire (pts (xy 20.32 15.24) (xy 20.32 72.39))
     (stroke (width 0) (type default) (color 0 0 0 0))
   )
@@
     (stroke (width 0) (type default) (color 0 0 0 0))
   )
-  (wire (pts (xy 27.94 72.39) (xy 17.78 72.39))
-    (stroke (width 0) (type default) (color 0 0 0 0))
-  )
   (wire (pts (xy 152.4 80.01) (xy 152.4 88.9))
     (stroke (width 0) (type default) (color 0 0 0 0))
@@
   )
   (wire (pts (xy 165.1 77.47) (xy 177.8 77.47))
-    (stroke (width 0) (type default) (color 0 0 0 0))
-  )
-  (wire (pts (xy 27.94 72.39) (xy 27.94 87.63))
     (stroke (width 0) (type default) (color 0 0 0 0))
   )
@@
     (pin "1")
     (pin "2")
-  )
-  (symbol (lib_id "Connector:Screw_Terminal_01x04") (at 12.7 69.85 0) (mirror y) (unit 1)
-    (in_bom yes) (on_board yes)
-    (property "Reference" "J1" (id 0) (at 14.7828 80.645 0))
-    (property "Value" "Screw_Terminal_01x04" (id 1) (at 14.7828 78.3336 0))
-    (property "Footprint" "TerminalBlock:TerminalBlock_Altech_AK300-4_P5.00mm" (id 2) (at 12.7 69.85 0)
-      (effects (font (size 1.27 1.27)) hide)
-    )
-    (property "Datasheet" "~" (id 3) (at 12.7 69.85 0)
-      (effects (font (size 1.27 1.27)) hide)
-    )
-    (pin "1")
-    (pin "2")
-    (pin "3")
-    (pin "4")
   )
   (symbol (lib_id "Transistor_BJT:BC847") (at 237.49 73.66 0) (unit 1)
@@
     (pin "1")
   )
+  (symbol (lib_id "Connector:Screw_Terminal_01x03") (at 12.7 69.85 0) (mirror y) (unit 1)
+    (in_bom yes) (on_board yes)
+    (property "Reference" "J1" (id 0) (at 10.668 68.7832 0)
+      (effects (font (size 1.27 1.27)) (justify left))
+    )
+    (property "Value" "Screw_Terminal_01x03" (id 1) (at 10.668 71.0946 0)
+      (effects (font (size 1.27 1.27)) (justify left))
+    )
+    (property "Footprint" "TerminalBlock:TerminalBlock_Altech_AK300-3_P5.00mm" (id 2) (at 12.7 69.85 0)
+      (effects (font (size 1.27 1.27)) hide)
+    )
+    (property "Datasheet" "~" (id 3) (at 12.7 69.85 0)
+      (effects (font (size 1.27 1.27)) hide)
+    )
+    (pin "1")
+    (pin "2")
+    (pin "3")
+  )
   (symbol (lib_id "Connector:Conn_01x06_Female") (at 195.58 115.57 0) (unit 1)
     (in_bom yes) (on_board yes) (fields_autoplaced)
@@
       (reference "D4") (unit 1) (value "1N4007") (footprint "Diode_SMD:D_SOD-123")
     )
-    (path "/00000000-0000-0000-0000-000061a48a61"
-      (reference "J1") (unit 1) (value "Screw_Terminal_01x04") (footprint "TerminalBlock:TerminalBlock_Altech_AK300-4_P5.00mm")
+    (path "/62009989-8103-49af-b226-a7bac174e878"
+      (reference "J1") (unit 1) (value "Screw_Terminal_01x03") (footprint "TerminalBlock:TerminalBlock_Altech_AK300-3_P5.00mm")
     )
     (path "/00000000-0000-0000-0000-0000616d5b91"
